File: pcb/Analog_Front_End/AFE.kicad_sch (KiCad schematic)
At the start: 16 parts, among them U1 TLV3603DCKR, U2 LM393

Commit message: various changes, including power, channel logic, FPGA
Parts:
- removed C2: ??? pF, symbol Device:C_Small
- added C2: JZ100, symbol Device:C_Trim_Small
- added C5: 100nF, symbol Device:C_Small
- added R10: 33, symbol Device:R_Small_US
- C1: value ??? pF -> 10pF
Connections:
- net CH1_EN is gone; now on net CH1_FA_N: U1.5 (LE/HYS)
- net 3V3: now also C5.1
- net CH1_CMP_IN: now also C2.1
- net CH1_OUT: now also R10.2; no longer U1.1 (OUT)
- net GND: now also C2.2, C5.2
- new net: R10.1, U1.1 (OUT)
Other:
- note added: "0.05pF"
- note added: "1pF"
- note added: "2-10pF"
- note added: "2pF"
- moved on the sheet: C3, R3, R4, R5, R6, R7, R8, R9, U1, U2A, U2B, U2C
