File: pcb/Analog_Front_End/Analog_Front_End.kicad_sch (KiCad schematic)
At the start: 0 parts

Commit message: various changes, including power, channel logic, FPGA
Other:
- added sheet FPGA (FPGA.kicad_sch)
Changed lines of the file:
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@@
+		)
+	)
+	(sheet
+		(at 70.485 85.09)
+		(size 62.865 27.94)
+		(exclude_from_sim no)
+		(in_bom yes)
+		(on_board yes)
+		(dnp no)
+		(fields_autoplaced yes)
+		(stroke
+			(width 0.1524)
+			(type solid)
+		)
+		(fill
+			(color 0 0 0 0)
+		)
+		(property "Sheetname" "FPGA"
+			(at 70.485 84.3784 0)
+			(show_name no)
+			(do_not_autoplace no)
+			(effects
+				(font
+					(size 1.27 1.27)
+				)
+				(justify left bottom)
+			)
+		)
+		(property "Sheetfile" "FPGA.kicad_sch"
+			(at 70.485 113.6146 0)
+			(show_name no)
+			(do_not_autoplace no)
+			(effects
+				(font
+					(size 1.27 1.27)
+				)
+				(justify left top)
+			)
+		)
+		(instances
+			(project "Analog_Front_End"
+				(path "/4f54a6ff-ef95-49cf-8ec8-d37622e08520"
+					(page "4")
+				)
+			)
 		)
 	)
