File: pcb/Analog_Front_End/PWR.kicad_sch (KiCad schematic)
At the start: 0 parts

Commit message: various changes, including power, channel logic, FPGA
Parts:
- added C4: 10uF, symbol Device:C_Small
- added C6, C7, C8: 100nF, symbol Device:C_Small
- added F1: 200mA Hold, 500mA Trip, symbol Device:Polyfuse
- added J1: USB_C_Receptacle_USB2.0_16P, symbol Connector:USB_C_Receptacle_USB2.0_16P
- added R11, R12: 5.1k, symbol Device:R_Small_US
- added S1: EG1213, EG1213:SW_EG1213, symbol Logic_Analyzer_AFE:EG1213
- added U3: AD5624RBRMZ-5REEL7, RM_10_ADI, symbol Logic_Analyzer_AFE:AD5624RBRMZ-5REEL7
- added U4: AP2112K-3.3, Package_TO_SOT_SMD:SOT-23-5, symbol Regulator_Linear:AP2112K-3.3
- added U5: AP2112K-2.5, Package_TO_SOT_SMD:SOT-23-5, symbol Regulator_Linear:AP2112K-2.5
Connections:
- new net: F1.1, J1.A4 (VBUS), J1.A9 (VBUS), J1.B4 (VBUS), J1.B9 (VBUS)
- new net: J1.A5 (CC1), R11.2
- new net: J1.B5 (CC2), R12.2
- new net 2V5: U5.5 (VOUT)
- new net 2V5_EN: U5.3 (EN)
- new net 3V3: C8.1, U4.5 (VOUT), U5.1 (VIN)
- new net 3V3_EN: U4.3 (EN)
- new net 5V: C4.1, C6.1, C7.1, S1.2, U3.9 (VDD), U4.1 (VIN)
- new net CH1_DAC_REF: U3.1 (VOUTA), U3.2 (VOUTB), U3.4 (VOUTC), U3.5 (VOUTD)
- new net DAC_CS: U3.6 (*SYNC)
- new net DAC_MOSI: U3.8 (DIN)
- new net DAC_SCLK: U3.7 (SCLK)
- new net GND: C4.2, C6.2, C7.2, C8.2, J1.A1 (GND), J1.A12 (GND), J1.B1 (GND), J1.B12 (GND), J1.SH (SHIELD), R11.1, R12.1, U3.10 (VREFIN/VREFOUT), U3.3 (GND), U4.2 (GND), U5.2 (GND)
- new net VBUS: F1.2, S1.3
- new net VU: S1.1
- no-connect marks 0 -> 6
